File: schematics/kicad/Thesis Remake.kicad_sch (KiCad schematic)
At the start: 119 parts, among them J1 SJ2-35853B-SMT-TR, J2 Conn_01x18, J3 Conn_01x18, J4 Conn_01x01_Pin, J5 Conn_01x01_Pin, J6 Conn_01x01_Pin, J7 Conn_01x01_Pin, U1 CD4051B, U10 MCP6001-OT, U11 MCP6001-OT, U2 PCM5102, U5 RT9080-33GJ5, U6 LM2940CT-5.0_MOD, U7 TPA711, U8 LM2940CT-5.0_MOD, U9 MCP6001-OT

Commit message: Commits
Parts:
- removed 0V1: TestPoint, TestPoint:TestPoint_Pad_1.5x1.5mm, symbol Connector:TestPoint
- removed C_COUPLING_MUX1: 10nF, Capacitor_SMD:C_1206_3216Metric_Pad1.33x1.80mm_HandSolder, symbol Device:C_Small
- removed D3: D_Schottky, Diode_SMD:D_SOD-123F, symbol Device:D_Schottky
- removed JP1, JP2, JP4, JP5, JP6, JP7, JP8, JP9: Jumper_2_Open, Jumper:SolderJumper-2_P1.3mm_Open_Pad1.0x1.5mm, symbol Jumper:Jumper_2_Open
- removed R_COUPLING_AMPSTAGE2: 10K, Resistor_SMD:R_0805_2012Metric_Pad1.20x1.40mm_HandSolder, symbol Device:R
- removed R_COUPLING_AMPSTAGE3: 1K, Resistor_SMD:R_0805_2012Metric_Pad1.20x1.40mm_HandSolder, symbol Device:R
- removed R_LADDER_4, R_LADDER_5, R_LADDER_6, R_LADDER_7, R_LADDER_8: 1k, Resistor_SMD:R_0805_2012Metric_Pad1.20x1.40mm_HandSolder, symbol Device:R
- removed U1: CD4051B, Package_SO:SOIC-16_3.9x9.9mm_P1.27mm, symbol Analog_Switch:CD4051B
- added C_COUPLING_MUX2: 10nF, Capacitor_SMD:C_1206_3216Metric_Pad1.33x1.80mm_HandSolder, symbol Device:C_Small
- added Q1: MMBT7002K, Package_TO_SOT_SMD:SOT-23, symbol MMBT7002K:MMBT7002K
- added RG3: 470, Resistor_SMD:R_0805_2012Metric_Pad1.20x1.40mm_HandSolder, symbol Device:R
- added RL1: 5K, Resistor_SMD:R_0805_2012Metric_Pad1.20x1.40mm_HandSolder, symbol Device:R
- added S2: B3F-1000, B3F-1000:SW_B3F-1000, symbol B3F-1000:B3F-1000
- added U3: SN74LVC1G3157, Package_TO_SOT_SMD:SOT-23-6, symbol SN74LVC1G3157:SN74LVC1G3157
- CG1_PCM5102, CG2_PCM5102: OC_Mouser 81-GRM31BR72E223KW01 -> 581-KGM21ACG1C222FU
- CI_TPA711, C_INPUT_LDO2, C_INPUT_LDO3: OC_Mouser 581-KAF31ER71H474KU -> 581-08055C474K4Z2A
- C_INPUT_RT9080: OC_Mouser 81-GCM31CR70J226ME3L -> 581-12063C105K4Z4A
- C_INPUT_TPA2: value 100nF -> 0.1uF
- J1: OC_Mouser (none) -> 490-SJ2-35853BSMT-TR
- J2, J3: Comments No idea -> (none); OC_Mouser (none) -> SAM15207-ND
- R5, R6, R7: OC_Mouser 708-RNHT0805BTE10K0 -> 708-RNHT0805BTE2K05
- ROUTDACL1, ROUTDACR1: OC_Mouser 71-RCS0805470KJNEA -> 603-RT0805BRE07470RL
- R_LADDER_2, R_LADDER_3: Comments (none) -> Depends; OC_Mouser 594-MCU08050C3300FP5 -> (none)
- STATUS_LED2, STATUS_LED3: OC_Mouser 594-MCU08050C3300FP5 -> 593-LSM0805412V
- U10, U11, U9: OC_Mouser (none) -> 579-MCP6001UT-I/OT
- U6, U8: OC_Mouser 926-LM2940IMPX50NOPB -> 926-LM2940CT50LF01
Connections:
- net +3.75V is gone; now on net ADC: R_LADDER_3.1
- net +5V: now also C_COUPLING_MUX2.1, RL1.2, U3.5 (+)
- net +5V1: no longer R_LADDER_2.2
- net ADC: now also J3.5 (Pin_5), R_LADDER_2.1; no longer J3.1 (Pin_1)
- net BUFFEROUT: now also U3.3 (A)
- net GND: now also R_LADDER_3.2, S1.1, C_COUPLING_MUX2.2, Q1.2, S2.1, U3.2 (-); no longer S1.2, S1.3
- net HI_LO: now also RG3.1
- net OUTDACR: now also U3.4 (C); no longer C_GND_AMPSTAGE3.1
- net +15V_Diode: now reaches C_INPUT_LDO2.2, C_IN_+15V_2.1, U6.1 (IN)
- net +15V_Diode: now also C_INPUT_LDO3.2, C_IN_+15V_3.1, D5.1 (K), U8.1 (IN)
- net +3v3_ESP: now reaches J2.17 (Pin_17)
- net +3v3_ESP: now also R_LADDER_2.2
- net Poll_Button_2: now reaches J2.2 (Pin_2)
- net Poll_Button_2: now also S2.4
- removed net +4.375V: R_LADDER_2.1, R_LADDER_3.2
- net Poll Button renamed Poll_Button_1
- net Poll_Button_1: no longer S1.1
- new net: Q1.3, RL1.1, U3.6 (S)
- new net: Q1.1, RG3.2
- new net Filter: C_GND_AMPSTAGE3.1, U3.1 (B)
- no-connect marks 35 -> 29
Other:
- note added: "Bachelorarbeit TODO: - Fix software: research libraries, fix PlatformIO configuration - Bypassing switch from FilterIN to FilterOUT - Research wave generation on ESP32 - Consider enclosing the board - Research about study groups - Consider reworking the layout: - Change test pads - Swap filter IN and OUT Add: Analog multiplexer as bypass switch instead of mechanical one -> button One button: pres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"
- note added: "Button 1: - long press will switch between Bluetooth and Waveform mode - short press will cycle waveforms in Waveform mode - triple press will result in bypass toggle Button 2 (only active in Waveform mode): - short press will cycle through various frequencies LED 1: - TBD LED 2: - TBD LED 3: - TBD"
- note added: "Comments: - one polarity diode, output of the diode goes to each LDO - redo resistor ladder circuit, use 3.3V supplied as output by the ESP - replace the MUX with the sn74LVC1G3157 - insure supplying the MUX with 5V - add a level shifter between ESP HI_LO label and MUX like a MOSFET (MMBT7002K), see circuits (open collector) - I2S protocol for waveform generation - how can you generate them? PCM?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"
- note added: "HEADPHONE JACK"
- note added: "If the control input is low, B1 channel is selected. If the control input is high, B2 channel is selected. The device permits signals with amplitudes of up to VCC (peak) to be transmitted. Level Shifter: https://tinyurl.com/2c3ztudm The logic coming from HI_LO pin shall be inverted."
- note added: "Pins in code correspond to Silkscreen names. EX: const uint8_t I2S_SCK = 14; /* Audio data bit clock */ means DO/IO14 is used IO6,7,8,9,10,11 or Pins 6,7,11,12,13,14 shall be avoided."
- note added: "STATUS"
- note added: "The RT9080 supplies the DAC."
- note added: "The first LM2940 shall only supply the ESP32. Only one reverse protection diode is used for both LMs."
- note added: "The second LM2940 supplies the rest of the ICs."
- note added: "Various resistor values will be used to set the board number and bluetooth name, depending on what is the output voltage read by the ADC. The ADC of the ESP can at most read 2.5V (=4095)."
- note removed: "Bachelorarbeit TODO: - Fix software: research libraries, fix PlatformIO configuration - Bypassing switch from FilterIN to FilterOUT - Research wave generation on ESP32 - Consider enclosing the board - Add trace from P2 to P3 on the jack for Mono Audio - Research about study groups - Add another LDO - Consider reworking the layout: - Change test pads - Rework Supply Trace - Swap filter IN and OUT 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"
- note removed: "Pins in code correspond to, for example "IO7/SD0"-names EX: const uint8_t I2S_SCK = 14; /* Audio data bit clock */ means DO/IO14 is used you shall not use IO6,7,8,9,10,11 so pins 6,7,11,12,13,14"
- moved on the sheet: +3V3, +5V1, +5V2, BCK1, BUFFER_OUT1, D10, D11, D5, D7, D8, D9, DEBUG1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

Commit message: Commits
Other:
- note added: "Level shifter & MUX"
- moved on the sheet: Q1, RG3, RL1, U3

Commit message: Commits
Parts:
- C1_APS_PCM5102, C_COUPLING_AMPSTAGE1, C_GND_AMPSTAGE1, C_GND_AMPSTAGE2, C_GND_AMPSTAGE3, C_INPUT_TPA1, C_INPUT_TPA3, C_IN_+15V_2, C_IN_+15V_3, C_IN_AMPSTAGE1: OC_Mouser 581-KAF31GR71C106KU -> 581-1206YC106KAT4A
- D7, D8, D9: footprint LED_THT:LED_D2.0mm_W4.8mm_H2.5mm_FlatTop -> LED_SMD:LED_0805_2012Metric_Pad1.15x1.40mm_HandSolder
Changed lines of the file:
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@@
 			)
 		)
-		(property "OC_Mouser" "581-KAF31GR71C106KU"
+		(property "OC_Mouser" "581-1206YC106KAT4A"
 			(at 317.5 87.63 0)
 			(effects
@@
 			)
 		)
-		(property "OC_Mouser" "581-KAF31GR71C106KU"
+		(property "OC_Mouser" "581-1206YC106KAT4A"
 			(at 316.23 168.91 0)
 			(effects
@@
 			)
 		)
-		(property "OC_Mouser" "581-KAF31GR71C106KU"
+		(property "OC_Mouser" "581-1206YC106KAT4A"
 			(at 55.88 66.04 0)
 			(effects
@@
 			)
 		)
-		(property "Footprint" "LED_THT:LED_D2.0mm_W4.8mm_H2.5mm_FlatTop"
+		(property "Footprint" "LED_SMD:LED_0805_2012Metric_Pad1.15x1.40mm_HandSolder"
 			(at 74.93 369.57 0)
 			(effects
@@
 			)
 		)
-		(property "OC_Mouser" "581-KAF31GR71C106KU"
+		(property "OC_Mouser" "581-1206YC106KAT4A"
 			(at 317.5 57.15 0)
 			(effects
@@
 			)
 		)
-		(property "Footprint" "LED_THT:LED_D2.0mm_W4.8mm_H2.5mm_FlatTop"
+		(property "Footprint" "LED_SMD:LED_0805_2012Metric_Pad1.15x1.40mm_HandSolder"
 			(at 58.42 369.57 0)
 			(effects
@@
 			)
 		)
-		(property "OC_Mouser" "581-KAF31GR71C106KU"
+		(property "OC_Mouser" "581-1206YC106KAT4A"
 			(at 474.98 184.15 0)
 			(effects
@@
 			)
 		)
-		(property "OC_Mouser" "581-KAF31GR71C106KU"
+		(property "OC_Mouser" "581-1206YC106KAT4A"
 			(at 54.61 118.11 0)
 			(effects
@@
 			)
 		)
-		(property "OC_Mouser" "581-KAF31GR71C106KU"
+		(property "OC_Mouser" "581-1206YC106KAT4A"
 			(at 534.67 104.14 0)
 			(effects
@@
 			)
 		)
-		(property "Footprint" "LED_THT:LED_D2.0mm_W4.8mm_H2.5mm_FlatTop"
+		(property "Footprint" "LED_SMD:LED_0805_2012Metric_Pad1.15x1.40mm_HandSolder"
 			(at 41.91 369.57 0)
 			(effects
@@
 			)
 		)
-		(property "OC_Mouser" "581-KAF31GR71C106KU"
+		(property "OC_Mouser" "581-1206YC106KAT4A"
 			(at 316.23 138.43 0)
 			(effects
@@
 			)
 		)
-		(property "OC_Mouser" "581-KAF31GR71C106KU"
+		(property "OC_Mouser" "581-1206YC106KAT4A"
 			(at 213.36 106.68 0)
 			(effects
@@
 			)
 		)
-		(property "OC_Mouser" "581-KAF31GR71C106KU"
+		(property "OC_Mouser" "581-1206YC106KAT4A"
 			(at 364.49 68.58 0)
 			(effects

Commit message: Commits
Connections:
- net BUFFEROUT: now also U3.1 (B); no longer CI_TPA711.2, U3.3 (A)
- net OUTDACR: now also C_GND_AMPSTAGE3.1, U3.3 (A); no longer U3.4 (C)
- removed net Filter: C_GND_AMPSTAGE3.1, U3.1 (B)
- new net Bypass: CI_TPA711.2, U3.4 (C)
Changed lines of the file:
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@@
 	(wire
 		(pts
-			(xy 405.13 148.59) (xy 405.13 152.4)
-		)
-		(stroke
-			(width 0)
-			(type default)
-		)
-	)
-	(wire
-		(pts
 			(xy 494.03 111.76) (xy 506.73 111.76)
 		)
@@
 	(wire
 		(pts
-			(xy 309.88 57.15) (xy 314.96 57.15)
-		)
-		(stroke
-			(width 0)
-			(type default)
-		)
-	)
-	(wire
-		(pts
 			(xy 113.03 114.3) (xy 125.73 114.3)
 		)
@@
 	(wire
 		(pts
+			(xy 311.15 57.15) (xy 314.96 57.15)
+		)
+		(stroke
+			(width 0)
+			(type default)
+		)
+	)
+	(wire
+		(pts
 			(xy 499.11 102.87) (xy 500.38 102.87)
 		)
@@
 	)
 	(label "Bypass"
-		(at 279.4 267.97 180)
+		(at 307.34 262.89 0)
 		(effects
 			(font
 				(size 1.27 1.27)
 			)
-			(justify right bottom)
+			(justify left bottom)
 		)
 	)
@@
 		)
 	)
-	(label "Filter"
-		(at 279.4 262.89 180)
-		(effects
-			(font
-				(size 1.27 1.27)
-			)
-			(justify right bottom)
-		)
-	)
 	(label "Poll_Button_1"
 		(at 107.95 335.28 180)
@@
 		)
 	)
+	(label "BUFFEROUT"
+		(at 279.4 262.89 180)
+		(effects
+			(font
+				(size 1.27 1.27)
+			)
+			(justify right bottom)
+		)
+	)
 	(label "IN"
 		(at 528.32 156.21 0)
@@
 	)
 	(label "Bypass"
-		(at 405.13 148.59 0)
+		(at 474.98 156.21 180)
 		(effects
 			(font
 				(size 1.27 1.27)
 			)
-			(justify left bottom)
+			(justify right bottom)
 		)
 	)
@@
 		)
 	)
+	(label "OUTDACR"
+		(at 311.15 57.15 180)
+		(effects
+			(font
+				(size 1.27 1.27)
+			)
+			(justify right bottom)
+		)
+	)
 	(label "DGND"
 		(at 212.09 193.04 180)
@@
 	)
 	(label "OUTDACR"
-		(at 307.34 262.89 0)
+		(at 279.4 267.97 180)
 		(effects
 			(font
 				(size 1.27 1.27)
 			)
-			(justify left bottom)
+			(justify right bottom)
 		)
 	)
@@
 		)
 	)
-	(label "Filter"
-		(at 309.88 57.15 180)
-		(effects
-			(font
-				(size 1.27 1.27)
-			)
-			(justify right bottom)
-		)
-	)
 	(label "Filter_IN"
 		(at 398.78 68.58 0)
@@
 		(effects
 			(font
-				(size 1.27 1.27)
-			)
-			(justify right bottom)
-		)
-	)
-	(label "BUFFEROUT"
-		(at 474.98 156.21 180)
-		(effects
-			(font

Commit message: Commits
Parts:
- C1_APS_PCM5102, C_GND_AMPSTAGE1, C_GND_AMPSTAGE2, C_INPUT_TPA1, C_IN_+15V_2, C_IN_+15V_3: Comments (none) -> 16V, X7R, 1206; Description_1 (none) -> input/gnd
- C1_CPPS_PCM1, C1_DPS_PCM1, C2_APS_PCM5102, C2_DPS_PCM1, C_INPUT_TPA2, C_SE/BTL_TPA1: Comments 0.1uF = 100nF -> 50V, X7R, 1206, 0.1uF = 100nF; Description_1 (none) -> input/gnd
- C2_CPPS_PCM1, CA_PCM5102, CB_TPA1: Comments (none) -> 25V, X7R, 1206; Description_1 (none) -> decoupling, datasheet recommendation
- CF_TPA711: Comments (none) -> 100V, C0G, 1206; Description_1 (none) -> pole compensation, datasheet recommendation
- CG1_PCM5102, CG2_PCM5102: Comments (none) -> 16V, X7R, 1206; Description_1 (none) -> low pass, fc = 150kHz; OC_Mouser 581-KGM21ACG1C222FU -> 581-1206YC222KAT2A
- CI_TPA711, C_INPUT_LDO2, C_INPUT_LDO3: Comments (none) -> 50V, X7R, 1206; Description_1 (none) -> input/gnd
- C_COUPLING_AMPSTAGE1, C_GND_AMPSTAGE3, C_INPUT_TPA3, C_IN_AMPSTAGE1: Comments (none) -> 16V, X7R, 1206; Description_1 (none) -> DC decoupling
- C_COUPLING_AMPSTAGE2, C_COUPLING_AMPSTAGE3, C_COUPLING_AMPSTAGE4, C_COUPLING_MUX2: Comments (none) -> 10V, X7R, 1206; Description_1 (none) -> input/gnd; OC_Mouser 581-KGM31GCG2J103JU -> 581-1206ZC103KAT2A
- C_INPUT_RT1, C_OUTPUT_LDO2, C_OUTPUT_LDO3: Description_1 (none) -> regulation during transients, datasheet recommendation
- C_INPUT_RT9080: Description_1 (none) -> input.gnd
- R1, R2, R3, R4, RI_TPA711: OC_Mouser 708-RNHT0805BTE10K0 -> 603-RC0805FR-0710KL; Replacement Part (none) -> 603-RC0805FR-0710KL
- R11: OC_Mouser 652-CR0805AFX1001EAS -> 603-RC0805FR-071KL; Replacement Part (none) -> 603-RC0805FR-071KL
- R12, R13, RG2, R_COUPLING_AMPSTAGE1: OC_Mouser 603-RT0805BRE07100KL -> 603-RC0805FR-07100KL; Replacement Part (none) -> 603-RC0805FR-07100KL
- R5, R6, R7: OC_Mouser 708-RNHT0805BTE2K05 -> 603-RC0805FR-072K2L; Replacement Part (none) -> 603-RC0805FR-072K2L
- RF1, RF2, RL1: OC_Mouser 71-RCA08055K10FKEA -> 603-RC0805FR-075K1L; Replacement Part (none) -> 603-RC0805FR-075K1L

Commit message: code commits
Parts:
- removed C_COUPLING_AMPSTAGE4: 10nF, Capacitor_SMD:C_1206_3216Metric_Pad1.33x1.80mm_HandSolder, symbol Device:C_Small
- removed C_INPUT_LDO2: 0.47uF, Capacitor_SMD:C_1206_3216Metric_Pad1.33x1.80mm_HandSolder, symbol Device:C_Small
- removed C_INPUT_RT1, C_OUTPUT_LDO2: 22uF, Capacitor_SMD:C_1206_3216Metric_Pad1.33x1.80mm_HandSolder, symbol Device:C_Small
- removed C_IN_+15V_2: 10uF, Capacitor_SMD:C_1206_3216Metric_Pad1.33x1.80mm_HandSolder, symbol Device:C_Small
- removed STATUS_LED2: 330, Resistor_SMD:R_0805_2012Metric_Pad1.20x1.40mm_HandSolder, symbol Device:R
- added C23: 10nF, Capacitor_SMD:C_1206_3216Metric_Pad1.33x1.80mm_HandSolder, symbol Device:C_Small
- added C4: 10uF, Capacitor_SMD:C_1206_3216Metric_Pad1.33x1.80mm_HandSolder, symbol Device:C_Small
- added C5: 0.47uF, Capacitor_SMD:C_1206_3216Metric_Pad1.33x1.80mm_HandSolder, symbol Device:C_Small
- added C6, C8: 22uF, Capacitor_SMD:C_1206_3216Metric_Pad1.33x1.80mm_HandSolder, symbol Device:C_Small
- added R2: 330, Resistor_SMD:R_0805_2012Metric_Pad1.20x1.40mm_HandSolder, symbol Device:R
- C12: renamed from C2_APS_PCM5102; Comments 50V, X7R, 1206, 0.1uF = 100nF -> 50V, X7R, 1206, 0.1uF = 100nF, C1206C104K3RAC7411
- C13: renamed from C1_CPPS_PCM1; Comments 50V, X7R, 1206, 0.1uF = 100nF -> 50V, X7R, 1206, 0.1uF = 100nF, C1206C104K3RAC7411
- C15: renamed from C1_DPS_PCM1; Comments 50V, X7R, 1206, 0.1uF = 100nF -> 50V, X7R, 1206, 0.1uF = 100nF, C1206C104K3RAC7411
- C16: renamed from C2_DPS_PCM1; Comments 50V, X7R, 1206, 0.1uF = 100nF -> 50V, X7R, 1206, 0.1uF = 100nF, C1206C104K3RAC7411
- C2: renamed from C_INPUT_LDO3; OC_Mouser 581-08055C474K4Z2A -> 80-C1206C474K4R
- C26: renamed from C_SE/BTL_TPA1; Comments 50V, X7R, 1206, 0.1uF = 100nF -> 50V, X7R, 1206, 0.1uF = 100nF, C1206C104K3RAC7411
- C28: renamed from C_INPUT_TPA2; Comments 50V, X7R, 1206, 0.1uF = 100nF -> 50V, X7R, 1206, 0.1uF = 100nF, C1206C104K3RAC7411
- C3: renamed from C_OUTPUT_LDO3; Comments (none) -> 6.3 VDC, 22uF, 1206, X7R; OC_Mouser 81-GCM31CR70J226ME3L -> 963-LMK316ABJ226MLHT
- C33: renamed from CI_TPA711; OC_Mouser 581-08055C474K4Z2A -> 80-C1206C474K4R
- C7: renamed from C_INPUT_RT9080; Comments (none) -> 25V, X7R, 1206; OC_Mouser 581-12063C105K4Z4A -> 80-C1206C105M3R
- R1: renamed from STATUS_LED3; OC_Mouser 593-LSM0805412V -> 603-RT0805BRE07470RL
- renumbered C_IN_+15V_3 to C1, CG2_PCM5102 to C10, C1_APS_PCM5102 to C11, C2_CPPS_PCM1 to C14, C_GND_AMPSTAGE3 to C17, C_COUPLING_AMPSTAGE2 to C18, C_COUPLING_AMPSTAGE1 to C19, C_GND_AMPSTAGE1 to C20, C_IN_AMPSTAGE1 to C21, C_COUPLING_AMPSTAGE3 to C22, C_GND_AMPSTAGE2 to C24, CB_TPA1 to C25, C_INPUT_TPA1 to C27, CF_TPA711 to C29, C_INPUT_TPA3 to C30, C_COUPLING_MUX2 to C31, CA_PCM5102 to C32, CG1_PCM5102 to C9, R3 to R10, R4 to R11, RG2 to R12, RF2 to R13, R13 to R14, R12 to R15, RF_TPA711 to R16, RI_TPA711 to R17, R11 to R18, RL1 to R19, RG3 to R20, R_LADDER_2 to R21, R_LADDER_3 to R22, R5 to R23, R6 to R24, R7 to R25, ROUTDACL1 to R3, ROUTDACR1 to R4, R1 to R5, R2 to R6, RG1 to R7, RF1 to R8, R_COUPLING_AMPSTAGE1 to R9, TP_VCC_AS2 to VCC_AS2, TP_VCC_Buffer1 to VCC_Buffer1
Connections:
- net +15V_Diode: now also C4.1, C5.2
- net +3v3: now also C8.2
- net +5V: now also C23.2
- net +5V1: now also C6.2
- net GND: now also C23.1, C4.2, C5.1, C6.1, C8.1, R2.1
- net at D11.1 (K): now also R2.2
Other:
- moved on the sheet: +5V1, D10, D5, U8, VCC_AS1, VCC_AS2, VCC_Buffer1

Commit message: Bluetooth works. Waveform generation glitches due to continuous generation.
Other:
- note added: "Bachelorarbeit TODO: - Fix software: research libraries, fix PlatformIO configuration - Consider enclosing the board - Research about study groups"
- note added: "TODO for next iteration: - move buttons more on the right side - change the TX pinned button to IO27 - add an external RST"
- note removed: "Bachelorarbeit TODO: - Fix software: research libraries, fix PlatformIO configuration - Bypassing switch from FilterIN to FilterOUT - Research wave generation on ESP32 - Consider enclosing the board - Research about study groups - Consider reworking the layout: - Change test pads - Swap filter IN and OUT Add: Analog multiplexer as bypass switch instead of mechanical one -> button One button: pres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"
- note removed: "Comments: - one polarity diode, output of the diode goes to each LDO - redo resistor ladder circuit, use 3.3V supplied as output by the ESP - replace the MUX with the sn74LVC1G3157 - insure supplying the MUX with 5V - add a level shifter between ESP HI_LO label and MUX like a MOSFET (MMBT7002K), see circuits (open collector) - I2S protocol for waveform generation - how can you generate them? PCM?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"
Changed lines of the file:
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@@
 		)
 	)
-	(text "Bachelorarbeit TODO:\n\n- Fix software: research libraries, fix PlatformIO configuration\n- Bypassing switch from FilterIN to FilterOUT\n- Research wave generation on ESP32\n- Consider enclosing the board\n- Research about study groups\n- Consider reworking the layout:\n	- Change test pads\n	- Swap filter IN and OUT\n\nAdd: \nAnalog multiplexer as bypass switch instead of mechanical one -> button\nOne button: pressing it fast will cycle waveforms, longpress will start bluetooth mode\nled for pairing and waveform, another led for bypass switch, test led for on/off\n\nModes:\n- long press = bluetooth on/off\n- short press 1 = sine\n- short press 1 = square\n- short press 1 = saw\n"
+	(text "Bachelorarbeit TODO:\n\n- Fix software: research libraries, fix PlatformIO configuration\n- Consider enclosing the board\n- Research about study groups\n"
 		(exclude_from_sim no)
-		(at -176.022 36.83 0)
+		(at 444.5 317.246 0)
 		(effects
 			(font
@@
 		)
 	)
+	(text "TODO for next iteration: \n- move buttons more on the right side \n- change the TX pinned button to IO27\n- add an external RST "
+		(exclude_from_sim no)
+		(at 445.77 340.868 0)
+		(effects
+			(font
+				(size 2.54 2.54)
+				(thickness 0.508)
+				(bold yes)
+				(color 29 42 255 1)
+			)
+			(justify left)
+		)
+	)
 	(text "The first LM2940 shall only supply the ESP32.\n\nOnly one reverse protection diode is used for both LMs."
 		(exclude_from_sim no)
@@
 		)
 	)
-	(text "Comments:\n- one polarity diode, output of the diode\ngoes to each LDO\n- redo resistor ladder circuit, use 3.3V supplied as output by the ESP\n- replace the MUX with the sn74LVC1G3157\n- insure supplying the MUX with 5V\n- add a level shifter between ESP HI_LO label and MUX like a MOSFET (MMBT7002K), see circuits (open collector)\n- I2S protocol for waveform generation - how can you generate them? PCM? \n- ESD protection by adding 1k after bias node and noninverting input of 2nd MCP6001"
-		(exclude_from_sim no)
-		(at -176.276 -31.75 0)
-		(effects
-			(font
-				(size 2.54 2.54)
-				(thickness 0.508)
-				(bold yes)
-				(color 0 255 0 1)
-			)
-			(justify left)
-		)
-	)
 	(text "DIGITAL POWER SUPPLY\n"
 		(exclude_from_sim no)
@@
 			"AAAAAAAAAAAAAAAAAAAAAAAAAAAAAAAAAAAAAAAAAAAAAAAAAAAAAAAAAAAAAAAAAAAAAAAAAAAA"
 			"AAAAAAAAAAAAAAAAAAAAAAAAAAAAAAAAAAAAAAAAAAAAAAAAAAAAAAAAAAAAAAAAAAAAAAAAAAAA"
+			"AAAAAAAAAAAAAAAAAAAAAAAAAAAAAAAAAAAAAAAAAAAAAAAAAAAAAAAAAAAAAAAAAAAAAAAAAAAA"
+			"AAAAAAAAAAAAAAAAAAAAAAAAAAAAAAAAAAAAAAAAAAAAAAAAAAAAAAAAAAAAAAAAAAAAAAAAAAAA"
+			"AAAAAAAAAAAAAAAAAAAAAAAAAAAAAAAAAAAAAAAAAAAAAAAAAAAAAAAAAAAAAAAAAAAAAAAAAAAA"
+			"AAAAAAAAAAAAAAAAAAAAAAAAAAAAAAAAAAAAAAAAAAAAAAAAAAAAAAAAAAAAAAAAAAAAAAAAAAAA"
+			"AAAAAAAAAAAAAAAAAAAAAAAAAAAAAAAAAAAAAAAAAAAAAAAAAAAAAAAAAAAAAAAAAAAAAAAAAAAA"
+			"AAAAAAAAAAAAAAAAAAAAAAAAAAAAAAAAAAAAAAAAAAAAAAAAAAAAAAAAAAAAAAAAAAAAAAAAAAAA"
+			"AAAAAAAAAAAAAAAAAAAAAAAAAAAAAAAAAAAAAAAAAAAAAAAAAAAAAAAAAAAAAAAAAAAAAAAAAAAA"
+			"AAAAAAAAAAAAAAAAAAAAAAAAAAAAAAAAAAAAAAAAAAAAAAAAAAAAAAAAAAAAAAAAAAAAAAAAAAAA"
+			"AAAAAAAAAAAAAAAAAAAAAAAAAAAAAAAAAAAAAAAAAAAAAAAAAAAAAAAAAAAAAAAAAAAAAAAAAAAA"
+			"AAAAAAAAAAAAAAAAAAAAAAAAAAAAAAAAAAAAAAAAAAAAAAAAAAAAAAAAAAAAAAAAAAAAAAAAAAAA"
+			"AAAAAAAAAAAAAAAAAAAAAAAAAAAAAAAAAAAAAAAAAAAAAAAAAAAAAAAAAAAAAAAAAAAAAAAAAAAA"
+			"AAAAAAAAAAAAAAAAAAAAAAAAAAAAAAAAAAAAAAAAAAAAAAAAAAAAAAAAAAAAAAAAAAAAAAAAAAAA"
+			"AAAAAAAAAAAAAAAAAAAAAAAAAAAAAAAAAAAAAAAAAAAAAAAAAAAAAAAAAAAAAAAAAAAAAAAAAAAA"
+			"AAAAAAAAAAAAAAAAAAAAAAAAAAAAAAAAAAAAAAAAAAAAAAAAAAAAAAAAAAAAAAAAAAAAAAAAAAAA"
+			"AAAAAAAAAAAAAAAAAAAAAAAAAAAAAAAAAAAAAAAAAAAAAAAAAAAAAAAAAAAAAAAAAAAAAAAAAAQA"
+			"AABadLcA8AAceUICAADwABx5QgIAAGAANxhCAgAAYAA3GEICAAAAQO0YQgIAAACwRgAAAAAAAAAA"
+			"AAAAAAAAAAAAAAAAAAAAAAAAAAAAAAAAAAAAAAAAAAAAAAAAAAAAAAAAAAAAAAAAAAAAAAAAAAAA"
+			"AAAAAAAAAAAAAAAAAAAAAAAAAAAAAAAAAAAAAAAAAAAAAAAAAAAAAAAAAAAAAAAAAAAAAAAAAAAA"
