File: schematics/kicad/Thesis Remake.kicad_sch (KiCad schematic)
At the start: 106 parts, among them J1 SJ2-35853B-SMT-TR, J2 Conn_01x18, J3 Conn_01x18, J4 Conn_01x01_Pin, J5 Conn_01x01_Pin, J6 Conn_01x01_Pin, J7 Conn_01x01_Pin, Q1 MMBT7002K, U10 MCP6001-OT, U11 MCP6001-OT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

Commit message: LUT Works now.
Parts:
- added C34: 10uF, Capacitor_SMD:C_1206_3216Metric_Pad1.33x1.80mm_HandSolder, symbol Device:C_Small
- added C35: 22uF, Capacitor_SMD:C_1206_3216Metric_Pad1.33x1.80mm_HandSolder, symbol Device:C_Small
- added PS1: TSR_0.5-2465, TSR_0.5-2465:CONV_TSR_0.5-2465, symbol TSR_0.5-2465:TSR_0.5-2465
- renumbered Vo+ to Vo+1, Vo- to Vo-1
Connections:
- net +15V_Diode: now also C34.1, PS1.1 (+VIN); no longer C4.1, C5.2, U6.1 (IN)
- net GND: now also C34.2, C35.1, PS1.2 (GND)
- new net +6.5V: C35.2, C4.1, C5.2, PS1.3 (+VOUT), U6.1 (IN)

Commit message: Commits
Parts:
- C35: Comments 6.3 VDC, 22uF, 1206, X7R -> 16V, X7R, 1206; Description_1 regulation during transients, datasheet recommendation -> input/gnd; OC_Mouser 963-LMK316ABJ226MLHT -> 581-1206YC106KAT4A
- Vo-1: footprint TestPoint:TestPoint_Pad_1.5x1.5mm -> TestPoint:TestPoint_Pad_2.5x2.5mm
Connections:
- net +6.5V: now also C35.1; no longer C35.2
- net GND: now also C35.2; no longer C35.1
Other:
- moved on the sheet: C34

Commit message: Reformatted code for easier reading.
Other:
- note added: "TODOs: - variable frequency ( cycle from 100 to x10Hz ) use short press of bypass button"
- note removed: "TODOs: Supply 1.1) Change LDO Package: I can test performance by using the TO-220 IC I have left from the Studienarbeit basket 1.2) Use DC-DC converter - could work, but since it's active switching, it could be noisy IO + HI/LO traces 2) Move buttons and HI_LO traces one pin lower, to avoid TX: I can test this by just retracing with a wire, like you have proposed Peripheral placement: 3) Move but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"
Changed lines of the file:
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@@
 		)
 	)
-	(text "TODOs:\n\nSupply\n1.1) Change LDO Package: I can test performance by using the TO-220 IC I have left from the Studienarbeit basket\n1.2) Use DC-DC converter - could work, but since it's active switching, it could be noisy\n\nIO + HI/LO traces\n2) Move buttons and HI_LO traces one pin lower, to avoid TX: I can test this by just retracing with a wire, like you have proposed\n\nPeripheral placement:\n3) Move buttons to be more accessible (more to the rightside edge of the board), which means lowering the speaker input block, and using a different audio jack package.\nI have used this package in my project with David: 179-SJ3-35052B. In my opinion, this package will alow some more space on that side of the board, making access to the two buttons easier. \nIt will also make plugging in and out of the PCB easier since it's perpendicular. What do you think?\n\n4) Populate 3rd LED - it will show if the signal is bypassed or not. This would add lots of visual aid.\n\n5) Make test pads larger, and silkscreen text also larger. I was thinking if there could be a way of soldering some upright wires to these test pads to make using the oscilloscope easier, by having the probes directly on the PCB.\n\nUse LED to indicate device state. You do not need a LED when the button is pressed....\nIncrease volume of build-in function generator to get a good noise floor.\nI added a DC/DC to the Mouser order so we can test the performance."
+	(text "TODOs: \n\n- variable frequency ( cycle from 100 to x10Hz ) \nuse short press of bypass button"
 		(exclude_from_sim no)
-		(at 11.43 -17.526 0)
+		(at 11.43 -16.002 0)
 		(effects
 			(font
@@
 			"AAAAAAAAAAAAAAAAAAAAAAAAAAAAAAAAAAAAAAAAAAAAAAAAAAAAAAAAAAAAAAAAAAAAAAAAAAAA"
 			"AAAAAAAAAAAAAAAAAAAAAAAAAAAAAAAAAAAAAAAAAAAAAAAAAAAAAAAAAAAAAAAAAAAAAAAAAAAA"
+			"AAAAAAAAAAAAAAAAAAAAAAAAAAAAAAAAAAAAAAAAAAAAAAAAAAAAAAAAAAAAAAAAAAAAAAAAAAAA"
+			"AAAAAAAAAAAAAAAAAAAAAAAAAAAAAAAAAAAAAAAAAAAAAAAAAAAAAAAAAAAAAAAAAAAAAAAAAAAA"
+			"AAAAAAAAAAAAAAAAAAAAAAAAAAAAAAAAAAAAAAAAAAAAAAAAAAAAAAAAAAAAAAAAAAAAAAAAAAAA"
+			"AAAAAAAAAAAAAAAAAAAAAAAAAAAAAAAAAAAAAAAAAAAAAAAAAAAAAAAAAAAAAAAAAAAAAAAAAAAA"
+			"AAAAAAAAAAAAAAAAAAAAAAAAAAAAAAAAAAAAAAAAAAAAAAAAAAAAAAAAAAAAAAAAAAAAAAAAAAAA"
+			"AAAAAAAAAAAAAAAAAAAAAAAAAAAAAAAAAAAAAAAAAAAAAAAAAAAAAAAAAAAAAAAAAAAAAAAAAAAA"
+			"AAAAAAAAAAAAAAAAAAAAAAAAAAAAAAAAAAAAAAAAAAAAAAAAAAAAAAAAAAAAAAAAAAAAAAAAAAAA"
+			"AAAAAAAAAAAAAAAAAAAAAAAAAAAAAAAAAAAAAAAAAAAAAAAAAAAAAAAAAAAAAAAAAAAAAAAAAAAA"
+			"AAAAAAAAAAAAAAAAAAAAAAAAAAAAAAAAAAAAAAAAAAAAAAAAAAAAAAAAAAAAAAAAAAAAAAAAAAAA"
+			"AAAAAAAAAAAAAAAAAAAAAAAAAAAAAAAAAAAAAAAAAAAAAAAAAAAAAAAAAAAAAAAAAAAAAAAAAAAA"
+			"AAAAAAAAAAAAAAAAAAAAAAAAAAAAAAAAAAAAAAAAAAAAAAAAAAAAAAAAAAAAAAAAAAAAAAAAAAAA"
+			"AAAAAAAAAAAAAAAAAAAAAAAAAAAAAAAAAAAAAAAAAAAAAAAAAAAAAAAAAAAAAAAAAAAAAAAAAAAA"
+			"AAAAAAAAAAAAAAAAAAAAAAAAAAAAAAAAAAAAAAAAAAAAAAAAAAAAAAAAAAAAAAAAAAAAAAAAAAAA"
+			"AAAAAAAAAAAAAAAAAAAAAAAAAAAAAAAAAAAAAAAAAAAAAAAAAAAAAAAAAAAAAAAAAAAAAAAAAAAA"
+			"AAAAAAAAAAAAAAAAAAAAAAAAAAAAAAAAAAAAAAAAAAAAAAAAAAAAAAAAAAAAAAAAAAAAAAAAAAAA"
+			"AAAAAAAAAAAAAAAAAAAAAAAAAAAAAAAAAAAAAAAAAAAAAAAAAAAAAAAAAAAAAAAAAAAAAAAAAAAA"
+			"AAAAAAAAAAAAAAAAAAAAAAAAAAAAAAAAAAAAAAAAAAAAAAAAAAAAAAAAAAAAAAAAAAAAAAAAAAAA"
+			"AAAAAAAAAAAAAAAAAAAAAAAAAAAAAAAAAAAAAAAAAAAAAAAAAAAAAAAAAAAAAAAAAAAAAAAAAAAA"
