File: schematics/kicad/_autosave-Thesis Remake.kicad_sch (KiCad schematic)
At the start: 106 parts, among them J1 SJ2-35853B-SMT-TR, J2 Conn_01x18, J3 Conn_01x18, J4 Conn_01x01_Pin, J5 Conn_01x01_Pin, J6 Conn_01x01_Pin, J7 Conn_01x01_Pin, Q1 MMBT7002K, U10 MCP6001-OT, U11 MCP6001-OT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

Commit message: QOL PCB changes
Parts:
- renumbered Vo+ to Vo+1, Vo- to Vo-1
Changed lines of the file:
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@@
 		(on_board yes)
 		(dnp no)
-		(property "Reference" "Vo-"
+		(property "Reference" "Vo-1"
 			(at 454.152 80.264 0)
 			(effects
@@
 			(project "Studienarbeit"
 				(path "/e1f471d3-f850-4433-b54a-c7e6f7857097"
-					(reference "Vo-")
+					(reference "Vo-1")
 					(unit 1)
 				)
@@
 		(on_board yes)
 		(dnp no)
-		(property "Reference" "Vo+"
+		(property "Reference" "Vo+1"
 			(at 468.376 80.518 0)
 			(effects
@@
 			(project "Studienarbeit"
 				(path "/e1f471d3-f850-4433-b54a-c7e6f7857097"
-					(reference "Vo+")
+					(reference "Vo+1")
 					(unit 1)
 				)

Commit message: Moved bypass switch from Pin 25 to 27 temp
Parts:
- renumbered Vo+1 to Vo+, Vo-1 to Vo-
Connections:
- net HI_LO: no longer J2.5 (Pin_5)
- net Poll_Button_1: no longer J2.4 (Pin_4)
- net Poll_Button_2: no longer J2.3 (Pin_3)
Changed lines of the file:
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@@
 	(wire
 		(pts
-			(xy 59.69 254) (xy 64.77 254)
+			(xy 54.61 251.46) (xy 59.69 251.46)
 		)
 		(stroke
@@
 	(wire
 		(pts
-			(xy 59.69 248.92) (xy 64.77 248.92)
+			(xy 54.61 254) (xy 59.69 254)
 		)
 		(stroke
@@
 	(wire
 		(pts
-			(xy 59.69 251.46) (xy 64.77 251.46)
+			(xy 54.61 248.92) (xy 59.69 248.92)
 		)
 		(stroke
@@
 			"AAAAAAAAAAAAAAAAAAAAAAAAAAAAAAAAAAAAAAAAAAAAAAAAAAAAAAAAAAAAAAAAAAAAAAAAAAAA"
 			"AAAAAAAAAAAAAAAAAAAAAAAAAAAAAAAAAAAAAAAAAAAAAAAAAAAAAAAAAAAAAAAAAAAAAAAAAAAA"
+			"AAAAAAAAAAAAAAAAAAAAAAAAAAAAAAAAAAAAAAAAAAAAAAAAAAAAAAAAAAAAAAAAAAAAAAAAAAAA"
+			"AAAAAAAAAAAAAAAAAAAAAAAAAAAAAAAAAAAAAAAAAAAAAAAAAAAAAAAAAAAAAAAAAAAAAAAAAAAA"
+			"AAAAAAAAAAAAAAAAAAAAAAAAAAAAAAAAAAAAAAAAAAAAAAAAAAAAAAAAAAAAAAAAAAAAAAAAAAAA"
+			"AAAAAAAAAAAAAAAAAAAAAAAAAAAAAAAAAAAAAAAAAAAAAAAAAAAAAAAAAAAAAAAAAAAAAAAAAAAA"
+			"AAAAAAAAAAAAAAAAAAAAAAAAAAAAAAAAAAAAAAAAAAAAAAAAAAAAAAAAAAAAAAAAAAAAAAAAAAAA"
+			"AAAAAAAAAAAAAAAAAAAAAAAAAAAAAAAAAAAAAAAAAAAAAAAAAAAAAAAAAAAAAAAAAAAAAAAAAAAA"
+			"AAAAAAAAAAAAAAAAAAAAAAAAAAAAAAAAAAAAAAAAAAAAAAAAAAAAAAAAAAAAAAAAAAAAAAAAAAAA"
+			"AAAAAAAAAAAAAAAAAAAAAAAAAAAAAAAAAAAAAAAAAAAAAAAAAAAAAAAAAAAAAAAAAAAAAAAAAAAA"
+			"AAAAAAAAAAAAAAAAAAAAAAAAAAAAAAAAAAAAAAAAAAAAAAAAAAAAAAAAAAAAAAAAAAAAAAAAAAAA"
+			"AAAAAAAAAAAAAAAAAAAAAAAAAAAAAAAAAAAAAAAAAAAAAAAAAAAAAAAAAAAAAAAAAAAAAAAAAAAA"
+			"AAAAAAAAAAAAAAAAAAAAAAAAAAAAAAAAAAAAAAAAAAAAAAAAAAAAAAAAAAAAAAAAAAAAAAAAAAAA"
+			"AAAAAAAAAAAAAAAAAAAAAAAAAAAAAAAAAAAAAAAAAAAAAAAAAAAAAAAAAAAAAAAAAAAAAAAAAAAA"
+			"AAAAAAAAAAAAAAAAAAAAAAAAAAAAAAAAAAAAAAAAAAAAAAAAAAAAAAAAAAAAAAAAAAAAAAAAAAAA"
+			"AAAAAAAAAAAAAAAAAAAAAAAAAAAAAAAAAAAAAAAAAAAAAAAAAAAAAAAAAAAAAAAAAAAAAAAAAAAA"
+			"AAAAAAAAAAAAAAAAAAAAAAAAAAAAAAAAAAAAAAAAAAAAAAAAAAAAAAAAAAAAAAAAAAAAAAAAAAAA"
+			"AAAAAAAAAAAAAAAAAAAAAAAAAAAAAAAAAAAAAAAAAAAAAAAAAAAAAAAAAAAAAAAAAAAAAAAAAAAA"
+			"AAAAAAAAAAAAAAAAAAAAAAAAAAAAAAAAAAAAAAAAAAAAAAAAAAAAAAAAAAAAAAAAAAAAAAAAAAAA"
+			"AAAAAAAAAAAAAAAAAAAAAAAAAAAAAAAAAAAAAAAAAAAAAAAAAAAAAAAAAAAAAAAAAAAAAAAAAAAA"
 			"AAAAAAAAAAAAAAAAAAAAAAAAAAAAAAAAAA=="
 		)
 	)
 	(label "Poll_Button_2"
-		(at 59.69 248.92 180)
+		(at 54.61 254 180)
 		(effects
 			(font
@@
 	)
 	(label "Poll_Button_1"
-		(at 59.69 251.46 180)
+		(at 54.61 248.92 180)
 		(effects
 			(font
@@
 	)
 	(label "HI_LO"
-		(at 59.69 254 180)
+		(at 54.61 251.46 180)
 		(effects
 			(font
@@
 		(on_board yes)
 		(dnp no)
-		(property "Reference" "Vo-1"
+		(property "Reference" "Vo-"
 			(at 454.152 80.264 0)
 			(effects
@@
 			(project "Studienarbeit"
 				(path "/e1f471d3-f850-4433-b54a-c7e6f7857097"
-					(reference "Vo-1")
+					(reference "Vo-")
 					(unit 1)
 				)
@@
 		(on_board yes)
 		(dnp no)
-		(property "Reference" "Vo+1"
+		(property "Reference" "Vo+"
 			(at 468.376 80.518 0)
 			(effects
@@
 			(project "Studienarbeit"
 				(path "/e1f471d3-f850-4433-b54a-c7e6f7857097"
-					(reference "Vo+1")
+					(reference "Vo+")
 					(unit 1)
 				)
