File: schematics/kicad/Thesis Remake.kicad_pcb (KiCad board)
At the start: 2 copper layers, 73 x 73 mm, 101 parts, among them J1 SJ2-35853B-SMT-TR, J2 Conn_01x18, J3 Conn_01x18, J4 Conn_01x01_Pin, J5 Conn_01x01_Pin, J6 Conn_01x01_Pin, J7 Conn_01x01_Pin, Q1 MMBT7002K, U10 MCP6001-OT, U11 MCP6001-OT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

Commit message: Added the TH Logo on the board.
Parts:
- added G***: LOGO, TH_MA_LOGO:TH_MA_Logo, F.Cu at (213.2, 64.8)
Other:
- board text added: "designed by: Paul Grămescu Prof. Simon Effler"
