File: schematics/kicad/Thesis Remake.kicad_pcb (KiCad board)
At the start: 2 copper layers, 73 x 73 mm, 102 parts, among them J1 SJ2-35853B-SMT-TR, J2 Conn_01x18, J3 Conn_01x18, J4 Conn_01x01_Pin, J5 Conn_01x01_Pin, J6 Conn_01x01_Pin, J7 Conn_01x01_Pin, Q1 MMBT7002K, U10 MCP6001-OT, U11 MCP6001-OT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

Commit message: Updated schematic in main
Parts:
- removed C35: 22uF, Capacitor_SMD:C_1206_3216Metric_Pad1.33x1.80mm_HandSolder
- removed U4: LM78M05_TO220, Package_TO_SOT_THT:TO-220-3_Vertical
- added PS1: TSR_0.5-2465, TSR_0.5-2465:CONV_TSR_0.5-2465, F.Cu at (208.8, 47.6)
- Vo-1: footprint TestPoint:TestPoint_Pad_1.5x1.5mm -> TestPoint:TestPoint_Pad_2.5x2.5mm
- moved C34 9.88 mm to (202.9, 40.5), turned to 90 degrees
- moved Vo-1 2.10 mm to (262.6, 65.4)
- moved LS1 0.83 mm to (268.9, 68.7)
- moved D5 0.52 mm to (213.9, 42.0)
- moved G*** 0.19 mm to (213.0, 64.9)
- moved D7 0.06 mm to (262.9, 50.5)
- renumbered BCK1 to BCK, DIN1 to DIN, LRCK1 to LRCK
Routing:
- net +6.5V: track 14.9 -> 17.8 mm
- net /Vo-: track 25.3 -> 26.4 mm
- net +15V_Diode: track 25.1 -> 26.0 mm
Other:
- board text added: "Bypass"
- board text added: "INPUT"
- board text added: "LED"
- board text added: "Mode"
- board text added: "No:"
- board text added: "OUTPUT"
- board text removed: "FILTER_IN"
- board text removed: "FILTER_OUT"
