File: schematics/kicad/_autosave-Thesis Remake.kicad_pcb (KiCad board)
At the start: 2 copper layers, 73 x 73 mm, 102 parts, among them J1 SJ2-35853B-SMT-TR, J2 Conn_01x18, J3 Conn_01x18, J4 Conn_01x01_Pin, J5 Conn_01x01_Pin, J6 Conn_01x01_Pin, J7 Conn_01x01_Pin, Q1 MMBT7002K, U10 MCP6001-OT, U11 MCP6001-OT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

Commit message: COmmits
Parts:
- moved C35 20.9 mm to (192.6, 43.5)
- moved C34 14.4 mm to (193.6, 40.4)
- moved U4 6.67 mm to (212.2, 46.6), turned to 180 degrees
Routing:
- net +15V_Diode: track 25.1 -> 11.9 mm
- net +6.5V: track 14.9 -> 5.26 mm
Other:
- board text added: "Bypass"
- board text added: "INPUT"
- board text added: "LED"
- board text added: "Mode"
- board text added: "OUTPUT"
- board text removed: "FILTER_IN"
- board text removed: "FILTER_OUT"
Changed lines of the file:
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@@
 	(footprint "Capacitor_SMD:C_1206_3216Metric_Pad1.33x1.80mm_HandSolder"
 		(layer "F.Cu")
-		(at 204.06 50.32 180)
+		(at 193.6225 40.35 180)
 		(descr "Capacitor SMD 1206 (3216 Metric), square (rectangular) end terminal, IPC_7351 nominal with elongated pad for handsoldering. (Body size source: IPC-SM-782 page 76, https://www.pcb-3d.com/wordpress/wp-content/uploads/ipc-sm-782a_amendment_1_and_2.pdf), generated with kicad-footprint-generator")
 		(tags "capacitor handsolder")
@@
 	(footprint "Capacitor_SMD:C_1206_3216Metric_Pad1.33x1.80mm_HandSolder"
 		(layer "F.Cu")
-		(at 212.32 50.36 180)
+		(at 192.62 43.53 180)
 		(descr "Capacitor SMD 1206 (3216 Metric), square (rectangular) end terminal, IPC_7351 nominal with elongated pad for handsoldering. (Body size source: IPC-SM-782 page 76, https://www.pcb-3d.com/wordpress/wp-content/uploads/ipc-sm-782a_amendment_1_and_2.pdf), generated with kicad-footprint-generator")
 		(tags "capacitor handsolder")
@@
 	(footprint "Package_TO_SOT_THT:TO-220-3_Vertical"
 		(layer "F.Cu")
-		(at 205.56 47.6)
+		(at 212.16 46.605 180)
 		(descr "TO-220-3, Vertical, RM 2.54mm, see https://www.vishay.com/docs/66542/to-220-1.pdf")
 		(tags "TO-220-3 Vertical RM 2.54mm")
@@
 		(attr through_hole)
 		(fp_line
-			(start -2.58 -3.27)
-			(end -2.58 1.371)
+			(start 7.66 -3.27)
+			(end 7.66 1.371)
 			(stroke
 				(width 0.12)
@@
 		)
 		(fp_line
-			(start -2.58 -3.27)
-			(end 7.66 -3.27)
+			(start 4.391 -3.27)
+			(end 4.391 -1.76)
 			(stroke
 				(width 0.12)
@@
 		)
 		(fp_line
-			(start -2.58 -1.76)
-			(end 7.66 -1.76)
+			(start 0.69 -3.27)
+			(end 0.69 -1.76)
 			(stroke
 				(width 0.12)
@@
 		)
 		(fp_line
-			(start 0.69 -3.27)
-			(end 0.69 -1.76)
+			(start -2.58 -1.76)
+			(end 7.66 -1.76)
 			(stroke
 				(width 0.12)
@@
 		)
 		(fp_line
-			(start 4.391 -3.27)
-			(end 4.391 -1.76)
+			(start -2.58 -3.27)
+			(end 7.66 -3.27)
 			(stroke
 				(width 0.12)
@@
 		)
 		(fp_line
-			(start 7.66 -3.27)
-			(end 7.66 1.371)
+			(start -2.58 -3.27)
+			(end -2.58 1.371)
 			(stroke
 				(width 0.12)
@@
 		)
 		(fp_line
-			(start -2.71 -3.4)
-			(end -2.71 1.51)
+			(start 7.79 1.51)
+			(end 7.79 -3.4)
 			(stroke
 				(width 0.05)
@@
 		)
 		(fp_line
-			(start -2.71 1.51)
-			(end 7.79 1.51)
+			(start 7.79 -3.4)
+			(end -2.71 -3.4)
 			(stroke
 				(width 0.05)
@@
 		)
 		(fp_line
-			(start 7.79 -3.4)
-			(end -2.71 -3.4)
+			(start -2.71 1.51)
+			(end 7.79 1.51)
 			(stroke
 				(width 0.05)
@@
 		)
 		(fp_line
-			(start 7.79 1.51)
-			(end 7.79 -3.4)
+			(start -2.71 -3.4)
+			(end -2.71 1.51)
 			(stroke
 				(width 0.05)
@@
 		)
 		(fp_line
-			(start -2.46 -3.15)
-			(end -2.46 1.25)
+			(start 7.54 1.25)
+			(end 7.54 -3.15)
 			(stroke
 				(width 0.1)
@@
 		)
 		(fp_line
-			(start -2.46 -1.88)
-			(end 7.54 -1.88)
+			(start 7.54 -3.15)
+			(end -2.46 -3.15)
 			(stroke
 				(width 0.1)
@@
 		)
 		(fp_line
-			(start -2.46 1.25)
-			(end 7.54 1.25)
+			(start 4.39 -3.15)
+			(end 4.39 -1.88)
 			(stroke
 				(width 0.1)
@@
 		)
 		(fp_line
-			(start 4.39 -3.15)
-			(end 4.39 -1.88)
+			(start -2.46 1.25)
+			(end 7.54 1.25)
 			(stroke
 				(width 0.1)
@@
 		)
 		(fp_line
-			(start 7.54 -3.15)
-			(end -2.46 -3.15)
+			(start -2.46 -1.88)
+			(end 7.54 -1.88)
 			(stroke
 				(width 0.1)
@@
 		)
 		(fp_line
-			(start 7.54 1.25)
-			(end 7.54 -3.15)
+			(start -2.46 -3.15)
+			(end -2.46 1.25)
 			(stroke
 				(width 0.1)
@@
 		)
 		(pad "1" thru_hole rect
-			(at 0 0)
+			(at 0 0 180)
 			(size 1.905 2)
 			(drill 1.1)
@@
 		)
 		(pad "2" thru_hole oval
-			(at 2.54 0)
+			(at 2.54 0 180)
 			(size 1.905 2)
 			(drill 1.1)
@@
 		)
 		(pad "3" thru_hole oval
-			(at 5.08 0)
+			(at 5.08 0 180)
 			(size 1.905 2)
 			(drill 1.1)
@@
 			(at 0 -1.648 0)
 			(layer "F.SilkS")
+			(hide yes)
 			(effects
 				(font
@@
 			(at 0 -1.648 0)
 			(layer "F.SilkS")
+			(hide yes)
 			(effects
 				(font
@@
 		(layer "Edge.Cuts")
 	)
-	(gr_text "FILTER_OUT"
-		(at 261.183333 34.72 0)
+	(gr_text "INPUT"
+		(at 262.91 34.72 0)
 		(layer "F.SilkS")
 		(effects
@@
 	)
 	(gr_text "GND"
-		(at 206.71 100.73 0)
+		(at 206.71 101.03 0)
 		(layer "F.SilkS")
 		(effects
@@
 		)
 	)
+	(gr_text "Bypass"
+		(at 255.411905 47.875 0)
+		(layer "F.SilkS")
+		(effects
+			(font
+				(size 1 1)
+				(thickness 0.1)
+			)
+			(justify left bottom)
+		)
+	)
+	(gr_text "Mode"
+		(at 256.95 62.89 0)
+		(layer "F.SilkS")
+		(effects
+			(font
+				(size 1 1)
+				(thickness 0.1)
+			)
+			(justify left bottom)
+		)
+	)
 	(gr_text "designed by:\nPaul Grămescu\nProf. Simon Effler\n"
 		(at 207.651657 72.31 0)
@@
 		)
 	)
-	(gr_text "FILTER_IN"
-		(at 261.85 100.73 0)
+	(gr_text "LED"
+		(at 256.65 51.26 0)
+		(layer "F.SilkS")
+		(effects
+			(font
+				(size 1 1)
+				(thickness 0.1)
+			)
+			(justify left bottom)
+		)
+	)
+	(gr_text "OUTPUT"
+		(at 262.44 101.03 0)
 		(layer "F.SilkS")
 		(effects
@@
 		)
 	)
+	(gr_text "Bypass\n"
+		(at 265.63 63.11 0)
+		(layer "F.SilkS")
+		(effects
+			(font
+				(size 1 1)
+				(thickness 0.1)
+			)
+			(justify left bottom)
+		)
+	)
+	(gr_text "Mode"
+		(at 256.102381 44.49 0)
+		(layer "F.SilkS")
+		(effects
+			(font
+				(size 1 1)
+				(thickness 0.1)
+			)
+			(justify left bottom)
+		)
+	)
 	(segment
 		(start 242.7375 36.2925)
@@
 	)
 	(segment
-		(start 205.56 47.6)
-		(end 205.58 47.58)
-		(width 1)
-		(layer "F.Cu")
-		(net 73)
-	)
-	(segment
-		(start 205.6225 50.32)
-		(end 205.555 50.2525)
-		(width 1)
-		(layer "F.Cu")
-		(net 73)
-	)
-	(segment
 		(start 214.81 43.14)
 		(end 214.81 42.07)
@@
 	)
 	(segment
-		(start 205.555 50.2525)
-		(end 205.555 47.605)
-		(width 1)
-		(layer "F.Cu")
-		(net 73)
-	)
-	(segment
 		(start 221.71625 38.98)
 		(end 221.73875 39.0025)
@@
 	)
 	(segment
-		(start 205.58 45.62)
-		(end 206.8 44.4)
-		(width 1)
-		(layer "F.Cu")
-		(net 73)
-	)
-	(segment
 		(start 215.79 39.85625)
 		(end 216.65125 38.995)
@@
 	)
 	(segment
-		(start 205.58 47.58)
-		(end 205.58 45.62)
-		(width 1)
-		(layer "F.Cu")
-		(net 73)
-	)
-	(segment
 		(start 213.55 44.4)
 		(end 214.81 43.14)
@@
 	)
 	(segment
-		(start 206.8 44.4)
-		(end 213.55 44.4)
-		(width 1)
-		(layer "F.Cu")
-		(net 73)
-	)
-	(segment
 		(start 216.65125 38.995)
 		(end 221.785 38.995)
@@
 	)
 	(segment
-		(start 205.555 47.605)
-		(end 205.56 47.6)
-		(width 1)
-		(layer "F.Cu")
-		(net 73)
-	)
-	(segment
 		(start 221.785 38.995)
 		(end 221.8 38.98)
@@
 	)
 	(segment
-		(start 210.7175 50.32)
-		(end 210.7175 47.6775)
-		(width 1)
-		(layer "F.Cu")
-		(net 84)
-	)
-	(segment
-		(start 210.7575 50.36)
-		(end 210.7175 50.32)
-		(width 1)
-		(layer "F.Cu")
-		(net 84)
-	)
-	(segment
-		(start 214.74 47.23)
-		(end 216.555 49.045)
-		(width 1)
-		(layer "F.Cu")
-		(net 84)
-	)
-	(segment
 		(start 221.765 49.045)
 		(end 221.79 49.07)
@@
 	)
 	(segment
-		(start 211.01 47.23)
-		(end 214.74 47.23)
-		(width 1)
-		(layer "F.Cu")
-		(net 84)
-	)
-	(segment
 		(start 216.555 49.045)
 		(end 221.765 49.045)
@@
 		(width 1)
 		(layer "F.Cu")
-		(net 84)
-	)
-	(segment
-		(start 210.7175 47.6775)
-		(end 210.64 47.6)
-		(width 1)
-		(layer "F.Cu")
-		(net 84)
-	)
-	(segment
-		(start 210.64 47.6)
-		(end 211.01 47.23)
-		(width 1)
-		(layer "F.Cu")
